Commit message: baxter with different T-pose

File: data/npc/baxter_description/urdf/baxter_edit.urdf (robot description, URDF)
Before this commit: robot baxter, 49 links, 48 joints
Joints:
- joint left_s0: origin xyz=0.055695 0 0.011038 rpy=0 0 0 -> xyz=0.055695 0 0.011038 rpy=0 0 0.5
- joint right_s0: origin xyz=0.055695 0 0.011038 rpy=0 0 0 -> xyz=0.055695 0 0.011038 rpy=0 0 -0.5

Commit message: baxter with different T-pose

File: data/npc/baxter_description/urdf/baxter_edit.urdf (robot description, URDF)
Before this commit: robot baxter, 49 links, 48 joints
Joints:
- joint left_e0: origin xyz=0.102 0 0 rpy=1.57079632679 -1.57079632679 1.57079632679 -> xyz=0.102 0 0 rpy=1.57079632679 1.57079632679 1.57079632679
- joint left_e0_fixed: origin xyz=0.107 0 0 rpy=1.57079632679 -1.57079632679 1.57079632679 -> xyz=0.107 0 0 rpy=1.57079632679 1.57079632679 1.57079632679
- joint right_e0: origin xyz=0.102 0 0 rpy=1.57079632679 1.57079632679 1.57079632679 -> xyz=0.102 0 0 rpy=1.57079632679 -1.57079632679 1.57079632679
- joint right_e0_fixed: origin xyz=0.107 0 0 rpy=1.57079632679 1.57079632679 1.57079632679 -> xyz=0.107 0 0 rpy=1.57079632679 -1.57079632679 1.57079632679
